Commit message: [y/n]!

File: src/jackal_description/urdf/accessories/vlp16_mount.urdf.xacro (robot description, xacro)
@@ -87,5 +87,9 @@
         <origin xyz="0 0 ${height}" rpy="0 0 0" />
       </joint>
-      <xacro:VLP-16 parent="${prefix}_vlp16_plate" topic="${topic}">
+<!--
+      <xacro:VLP-16 parent="${prefix}_vlp16_plate" topic="${topic} ">
+        <origin xyz="0 0 0" rpy="0 0 0" />
+      </xacro:VLP-16> -->
+      <xacro:VLP-16 parent="${prefix}_vlp16_plate" topic="${topic}" hz="50.0">
         <origin xyz="0 0 0" rpy="0 0 0" />
       </xacro:VLP-16>
